Commit message: show construct. cone and align_depth=true for color point cloud

File: urdf/_d435i.gazebo.xacro (robot description, xacro)
@@ -9,29 +9,29 @@
 -->
 <robot xmlns:xacro="http://ros.org/wiki/xacro">
-  <xacro:macro name="gazebo_d435i" params=" reference_link
-                                            camera_name:=camera
+  <xacro:macro name="gazebo_d435i" params=" camera_name:=camera
                                             topics_ns:=camera
+                                            reference_link
                                             depth_optical_frame
-                                            color_optical_frame
-                                            infrared1_optical_frame
-                                            infrared2_optical_frame
-                                            accel_optical_frame
-                                            gyro_optical_frame
-                                            visualize:=false
-                                            align_depth:=false
-                                            enable_pointCloud:=false
-                                            unite_imu_method:=false
-                                            accel_fps:=250
-                                            gyro_fps:=400
-                                            clip_distance:=-1.0
                                             depth_width:=1280
                                             depth_height:=720
                                             depth_fps:=30
+                                            color_optical_frame
+                                            color_width:=1920
+                                            color_height:=1080
+                                            color_fps:=30
+                                            infrared1_optical_frame
+                                            infrared2_optical_frame
                                             infra_width:=640
                                             infra_height:=480
                                             infra_fps:=30
-                                            color_width:=1920
-                                            color_height:=1080
-                                            color_fps:=30
+                                            accel_optical_frame
+                                            gyro_optical_frame
+                                            accel_fps:=250
+                                            gyro_fps:=400
+                                            enable_pointCloud:=false
+                                            unite_imu_method:=false
+                                            clip_distance:=-1.0
+                                            align_depth:=false
+                                            visualize:=false
                                             ">
     <!-- Load parameters to model's main link-->
@@ -249,5 +249,6 @@
       	<pointCloud>${enable_pointCloud}</pointCloud>
       	<pointCloudTopicName>depth/color/points</pointCloudTopicName>
-      	<pointCloudCutoff>0.5</pointCloudCutoff>
+        <!-- <pointCloudTopicName>depth_registered/points</pointCloudTopicName> -->
+      	<pointCloudCutoff>0.1</pointCloudCutoff>
       </plugin>
     </gazebo>

File: urdf/camera_belt.urdf.xacro (robot description, xacro)
@@ -3,6 +3,6 @@
   <link name="base_link"/>
   <!-- d435i frame definition can be found at https://github.com/IntelRealSense/librealsense/blob/master/doc/d435i.md -->
-  <xacro:include filename="$(find realsense_gazebo_description)/urdf/_d435i.urdf.xacro"/>
-  <xacro:sensor_d435i parent="base_link" name="D435i_camera" topics_ns="D435i_camera" visualize="true" enable_pointCloud="true" align_depth="true">
+  <xacro:include filename="$(find realsense_gazebo_description)/urdf/_d435i.urdf.xacro" />
+  <xacro:sensor_d435i parent="base_link" name="D435i_camera" topics_ns="D435i_camera" visualize="true" align_depth="true" enable_pointCloud="true">
     <origin xyz="0.0 0.0 0.0" rpy="0.0 0.0 0.0"/>
   </xacro:sensor_d435i>

File: urdf/multicamera.urdf.xacro (robot description, xacro)
@@ -14,10 +14,10 @@
   <!-- d435  frame definition can be found at https://github.com/IntelRealSense/librealsense/blob/master/doc/d435i.md -->
   <xacro:include filename="$(find realsense_gazebo_description)/urdf/_d435.urdf.xacro"/>
-  <xacro:sensor_d435  parent="base_link" name="D435_camera" topics_ns="D435_camera" visualize="true" enable_pointCloud="true">
+  <xacro:sensor_d435  parent="base_link" name="D435_camera" topics_ns="D435_camera" visualize="true" align_depth="true" enable_pointCloud="true">
     <origin xyz="0.0 -0.5 0.0" rpy="0.0 0.0 0.0"/>
   </xacro:sensor_d435>
   <!-- d435i frame definition can be found at https://github.com/IntelRealSense/librealsense/blob/master/doc/d435i.md -->
   <xacro:include filename="$(find realsense_gazebo_description)/urdf/_d435i.urdf.xacro"/>
-  <xacro:sensor_d435i parent="base_link" name="D435i_camera" topics_ns="D435i_camera" visualize="true" enable_pointCloud="true">
+  <xacro:sensor_d435i parent="base_link" name="D435i_camera" topics_ns="D435i_camera" visualize="true" align_depth="true" enable_pointCloud="true">
     <origin xyz="0.0 0.5 0.0" rpy="0.0 0.0 0.0"/>
   </xacro:sensor_d435i>
@@ -39,5 +39,7 @@
     <visual>
       <geometry>
-        <mesh filename="model://construction_cone/meshes/construction_cone.dae" scale="10 10 10"/>
+        <!-- <mesh filename="model://construction_cone/meshes/construction_cone.dae" scale="10 10 10"/> -->
+        <!-- export GAZEBO_MODEL_PATH=/home/user/.gazebo/models -->
+        <mesh filename="file://$(env GAZEBO_MODEL_PATH)/construction_cone/meshes/construction_cone.dae" scale="10 10 10"/>
       </geometry>
     </visual>

File: urdf/multicamera_params.urdf.xacro (robot description, xacro)
@@ -70,5 +70,7 @@
     <visual>
       <geometry>
-        <mesh filename="model://construction_cone/meshes/construction_cone.dae" scale="10 10 10"/>
+        <!-- <mesh filename="model://construction_cone/meshes/construction_cone.dae" scale="10 10 10"/> -->
+        <!-- export GAZEBO_MODEL_PATH=/home/user/.gazebo/models -->
+        <mesh filename="file://$(env GAZEBO_MODEL_PATH)/construction_cone/meshes/construction_cone.dae" scale="10 10 10"/>
       </geometry>
     </visual>

File: urdf/singlecamera_d435i.urdf.xacro (robot description, xacro)
@@ -4,5 +4,5 @@
   <!-- d435i frame definition can be found at https://github.com/IntelRealSense/librealsense/blob/master/doc/d435i.md -->
   <xacro:include filename="$(find realsense_gazebo_description)/urdf/_d435i.urdf.xacro"/>
-  <xacro:sensor_d435i parent="base_link" name="D435i_camera" topics_ns="D435i_camera" visualize="true" enable_pointCloud="true">
+  <xacro:sensor_d435i parent="base_link" name="D435i_camera" topics_ns="D435i_camera" align_depth="true" visualize="true" enable_pointCloud="true">
     <origin xyz="0.0 0.5 0.0" rpy="0.0 0.0 0.0"/>
   </xacro:sensor_d435i>
@@ -16,5 +16,7 @@
     <visual>
       <geometry>
-        <mesh filename="model://construction_cone/meshes/construction_cone.dae" scale="10 10 10"/>
+        <!-- <mesh filename="model://construction_cone/meshes/construction_cone.dae" scale="10 10 10"/> -->
+        <!-- export GAZEBO_MODEL_PATH=/home/user/.gazebo/models -->
+        <mesh filename="file://$(env GAZEBO_MODEL_PATH)/construction_cone/meshes/construction_cone.dae" scale="10 10 10"/>
       </geometry>
     </visual>

Commit message: (1) change pointCloudTopicName;(2)rviz

File: urdf/_d435i.gazebo.xacro (robot description, xacro)
@@ -248,7 +248,8 @@
         <!-- Pointlcloud settings -->
       	<pointCloud>${enable_pointCloud}</pointCloud>
-      	<pointCloudTopicName>depth/color/points</pointCloudTopicName>
-        <!-- <pointCloudTopicName>depth_registered/points</pointCloudTopicName> -->
-      	<pointCloudCutoff>0.1</pointCloudCutoff>
+        <pointCloudTopicName>depth_registered/points</pointCloudTopicName>
+        <!-- <pointCloudTopicName>depth/color/points</pointCloudTopicName> -->
+        <!-- <pointCloudTopicName>/camera/depth_registered/points</pointCloudTopicName> -->
+        <pointCloudCutoff>0.1</pointCloudCutoff>
       </plugin>
     </gazebo>

File: urdf/camera_belt.urdf.xacro (robot description, xacro)
@@ -4,5 +4,5 @@
   <!-- d435i frame definition can be found at https://github.com/IntelRealSense/librealsense/blob/master/doc/d435i.md -->
   <xacro:include filename="$(find realsense_gazebo_description)/urdf/_d435i.urdf.xacro" />
-  <xacro:sensor_d435i parent="base_link" name="D435i_camera" topics_ns="D435i_camera" visualize="true" align_depth="true" enable_pointCloud="true">
+  <xacro:sensor_d435i parent="base_link" name="camera" topics_ns="camera" visualize="true" align_depth="true" enable_pointCloud="true">
     <origin xyz="0.0 0.0 0.0" rpy="0.0 0.0 0.0"/>
   </xacro:sensor_d435i>
@@ -15,5 +15,5 @@
           <parent link="base_link"/>
           <child link="belt10mm_base_link"/>
-          <origin xyz="2 0.5 0" rpy="0 0 1.57"/>
+          <origin xyz="1 0.12 0" rpy="0 0 1.57"/>
   </joint>
   <!-- add a belt12mm -->
@@ -25,5 +25,5 @@
           <parent link="base_link"/>
           <child link="belt12mm_base_link"/>
-          <origin xyz="2 -0.5 0" rpy="0 0 1.57"/>
+          <origin xyz="1 -0.12 0" rpy="0 0 1.57"/>
   </joint>
 </robot>
