Commit message: [ok] visualize_color, clip_distance_z_min/max

File: urdf/_d435.gazebo.xacro (robot description, xacro)
@@ -16,5 +16,6 @@
                                           infrared1_optical_frame
                                           infrared2_optical_frame
-                                          clip_distance:=-1.0
+                                          clip_distance_z_min:=0.1
+                                          clip_distance_z_max:=-1.0
                                           depth_width:=1280
                                           depth_height:=720
@@ -131,9 +132,9 @@
           <clip>
             <near>0.1</near>
-            <xacro:unless value="${clip_distance > 0.0}">
+            <xacro:unless value="${clip_distance_z_max > 0.0}">
               <far>100</far>
             </xacro:unless>
-            <xacro:if value="${clip_distance > 0.0}">
-              <far>${clip_distance}</far>
+            <xacro:if value="${clip_distance_z_max > 0.0}">
+              <far>${clip_distance_z_max}</far>
             </xacro:if>
           </clip>
@@ -172,9 +173,9 @@
         <!-- Depth camera settings -->
       	<rangeMinDepth>0.2</rangeMinDepth>
-        <xacro:unless value="${clip_distance > 0.0}">
+        <xacro:unless value="${clip_distance_z_max > 0.0}">
       	  <rangeMaxDepth>10.0</rangeMaxDepth>
         </xacro:unless>
-        <xacro:if value="${clip_distance > 0.0}">
-          <rangeMaxDepth>${clip_distance}</rangeMaxDepth>
+        <xacro:if value="${clip_distance_z_max > 0.0}">
+          <rangeMaxDepth>${clip_distance_z_max}</rangeMaxDepth>
         </xacro:if>
         <xacro:unless value="${align_depth}">

File: urdf/_d435.urdf.xacro (robot description, xacro)
@@ -17,5 +17,6 @@
                                           align_depth:=false
                                           enable_pointCloud:=false
-                                          clip_distance:=-1.0
+                                          clip_distance_z_min:=0.1
+                                          clip_distance_z_max:=-1.0
                                           depth_width:=1280
                                           depth_height:=720
@@ -153,5 +154,6 @@
                         infra_fps="${infra_fps}"
                         enable_pointCloud="${enable_pointCloud}"
-                        clip_distance="${clip_distance}"
+                        clip_distance_z_min="${clip_distance_z_min}"
+                        clip_distance_z_max="${clip_distance_z_max}"
                         align_depth="${align_depth}"
                         visualize="${visualize}"

File: urdf/_d435i.gazebo.xacro (robot description, xacro)
@@ -20,4 +20,5 @@
                                             color_height:=1080
                                             color_fps:=30
+                                            visualize_color:=false
                                             infrared1_optical_frame
                                             infrared2_optical_frame
@@ -31,8 +32,8 @@
                                             enable_pointCloud:=false
                                             unite_imu_method:=false
-                                            clip_distance:=-1.0
+                                            clip_distance_z_min:=0.1
+                                            clip_distance_z_max:=-0.1
                                             align_depth:=false
-                                            visualize:=false
-                                            ">
+                                                                                        ">
     <!-- Load parameters to model's main link-->
     <xacro:property name="deg_to_rad" value="0.01745329251994329577"/>
@@ -51,4 +52,5 @@
       <!--<max_vel>0.01</max_vel>
       <min_depth>0</min_depth>-->
+      <!-- Color -->
       <sensor name="${camera_name}color" type="camera">
         <camera name="${camera_name}">
@@ -71,6 +73,7 @@
         <always_on>1</always_on>
         <update_rate>${color_fps}</update_rate>
-        <visualize>${visualize}</visualize>
-      </sensor>
+        <visualize>${visualize_color}</visualize>
+      </sensor>
+      <!-- InfarRed1:Left -->
       <sensor name="${camera_name}ired1" type="camera">
         <camera name="${camera_name}">
@@ -95,4 +98,5 @@
         <visualize>false</visualize>
       </sensor>
+      <!-- InfarRed2:Right -->
       <sensor name="${camera_name}ired2" type="camera">
         <camera name="${camera_name}">
@@ -117,4 +121,5 @@
         <visualize>false</visualize>
       </sensor>
+      <!-- Depth -->
       <sensor name="${camera_name}depth" type="depth">
         <camera name="${camera_name}">
@@ -135,10 +140,10 @@
           </xacro:if>
           <clip>
-            <near>0.1</near>
-            <xacro:unless value="${clip_distance > 0.0}">
+            <near>${clip_distance_z_min}</near>
+            <xacro:unless value="${clip_distance_z_max > 0.0}">
               <far>100</far>
             </xacro:unless>
-            <xacro:if value="${clip_distance > 0.0}">
-              <far>${clip_distance}</far>
+            <xacro:if value="${clip_distance_z_max > 0.0}">
+              <far>${clip_distance_z_max}</far>
             </xacro:if>
           </clip>
@@ -210,4 +215,5 @@
       </xacro:unless>
     </gazebo>
+    <!-- Load plugin to the model ("robot" in urdf format)-->
     <gazebo>
       <plugin name="${topics_ns}" filename="librealsense_gazebo_plugin.so">
@@ -228,9 +234,9 @@
         <!-- Depth camera settings -->
       	<rangeMinDepth>0.2</rangeMinDepth>
-        <xacro:unless value="${clip_distance > 0.0}">
+        <xacro:unless value="${clip_distance_z_max > 0.0}">
       	  <rangeMaxDepth>10.0</rangeMaxDepth>
         </xacro:unless>
-        <xacro:if value="${clip_distance > 0.0}">
-          <rangeMaxDepth>${clip_distance}</rangeMaxDepth>
+        <xacro:if value="${clip_distance_z_max > 0.0}">
+          <rangeMaxDepth>${clip_distance_z_max}</rangeMaxDepth>
         </xacro:if>
         <xacro:unless value="${align_depth}">

File: urdf/_d435i.urdf.xacro (robot description, xacro)
@@ -15,5 +15,5 @@
                                           name:=camera
                                           topics_ns:=camera
-                                          visualize:=false
+                                          visualize_color:=false
                                           align_depth:=false
                                           enable_pointCloud:=false
@@ -21,5 +21,6 @@
                                           accel_fps:=250
                                           gyro_fps:=400
-                                          clip_distance:=-1.0
+                                          clip_distance_z_min:=0.1
+                                          clip_distance_z_max:=-1.0
                                           depth_width:=1280
                                           depth_height:=720
@@ -187,7 +188,8 @@
                         enable_pointCloud="${enable_pointCloud}"
                         unite_imu_method="${unite_imu_method}"
-                        clip_distance="${clip_distance}"
+                        clip_distance_z_min="${clip_distance_z_min}"
+                        clip_distance_z_max="${clip_distance_z_max}"
                         align_depth="${align_depth}"
-                        visualize="${visualize}"
+                        visualize_color="${visualize_color}"
     />
   </xacro:macro>

File: urdf/camera_belt.urdf.xacro (robot description, xacro)
@@ -4,7 +4,12 @@
   <!-- d435i frame definition can be found at https://github.com/IntelRealSense/librealsense/blob/master/doc/d435i.md -->
   <xacro:include filename="$(find realsense_gazebo_description)/urdf/_d435i.urdf.xacro" />
-  <xacro:sensor_d435i parent="base_link" name="camera" topics_ns="camera" visualize="true" align_depth="true" enable_pointCloud="true">
+  <xacro:sensor_d435i parent="base_link" name="camera" topics_ns="camera" visualize_color="true" align_depth="true" enable_pointCloud="true">
     <origin xyz="0.0 0.0 0.0" rpy="0.0 0.0 0.0"/>
   </xacro:sensor_d435i>
+  <!-- d405 -->
+  <!-- <xacro:include filename="$(find realsense2_description)/urdf/_d405.urdf.xacro" />
+  <xacro:sensor_d405 parent="base_link" name="camera" topics_ns="camera" use_nominal_extrinsics="true" visualize_color="true" align_depth="true" enable_pointCloud="true">
+    <origin xyz="0.0 0.0 0.0" rpy="0.0 0.0 0.0"/>
+  </xacro:sensor_d405> -->
   <!-- add a belt10mm -->
   <xacro:include filename="$(find belt10mm_description)/urdf/belt10mm.xacro"/>

File: urdf/multicamera.urdf.xacro (robot description, xacro)
@@ -19,5 +19,5 @@
   <!-- d435i frame definition can be found at https://github.com/IntelRealSense/librealsense/blob/master/doc/d435i.md -->
   <xacro:include filename="$(find realsense_gazebo_description)/urdf/_d435i.urdf.xacro"/>
-  <xacro:sensor_d435i parent="base_link" name="D435i_camera" topics_ns="D435i_camera" visualize="true" align_depth="true" enable_pointCloud="true">
+  <xacro:sensor_d435i parent="base_link" name="D435i_camera" topics_ns="D435i_camera" visualize_color="true" align_depth="true" enable_pointCloud="true">
     <origin xyz="0.0 0.5 0.0" rpy="0.0 0.0 0.0"/>
   </xacro:sensor_d435i>

File: urdf/multicamera_params.urdf.xacro (robot description, xacro)
@@ -6,5 +6,6 @@
   <xacro:sensor_d435  parent="base_link" name="D435_camera" topics_ns="D435_camera"
                       enable_pointCloud="false"
-                      clip_distance="-1.0"
+                      clip_distance_z_min="0.1"
+                      clip_distance_z_max="-1.0"
                       align_depth="false"
                       visualize="false"
@@ -26,7 +27,8 @@
   <xacro:sensor_d435i parent="base_link" name="D435i_camera" topics_ns="D435i_camera"
                       enable_pointCloud="true"
-                      clip_distance="-1.0"
+                      clip_distance_z_min="-1.0"
+                      clip_distance_z_max="-1.0"
                       align_depth="false"
-                      visualize="false"
+                      visualize_color="false"
                       unite_imu_method="false"
                       accel_fps="250"

File: urdf/singlecamera_d435i.urdf.xacro (robot description, xacro)
@@ -4,5 +4,5 @@
   <!-- d435i frame definition can be found at https://github.com/IntelRealSense/librealsense/blob/master/doc/d435i.md -->
   <xacro:include filename="$(find realsense_gazebo_description)/urdf/_d435i.urdf.xacro"/>
-  <xacro:sensor_d435i parent="base_link" name="D435i_camera" topics_ns="D435i_camera" align_depth="true" visualize="true" enable_pointCloud="true">
+  <xacro:sensor_d435i parent="base_link" name="D435i_camera" topics_ns="D435i_camera" align_depth="true" visualize_color="true" enable_pointCloud="true">
     <origin xyz="0.0 0.5 0.0" rpy="0.0 0.0 0.0"/>
   </xacro:sensor_d435i>
