Commit message: add 2 belt

File: urdf/camera_belt.urdf.xacro (robot description, xacro)
@@ -7,4 +7,14 @@
     <origin xyz="0.0 0.0 0.0" rpy="0.0 0.0 0.0"/>
   </xacro:sensor_d435i>
+  <!-- add a belt10mm -->
+  <xacro:include filename="$(find belt10mm_description)/urdf/belt10mm.xacro"/>
+  <xacro:belt10mm parent="base_link" prefix="belt10mm_">
+    <origin xyz="0.0 0.0 0.0" rpy="0.0 0.0 0.0"/>
+  </xacro:belt10mm>
+  <joint name="belt10mm_joint" type="fixed">
+          <parent link="base_link"/>
+          <child link="belt10mm_base_link"/>
+          <origin xyz="2 0.5 0" rpy="0 0 1.57"/>
+  </joint>
   <!-- add a belt12mm -->
   <xacro:include filename="$(find belt12mm_description)/urdf/belt12mm.xacro"/>
@@ -15,5 +25,5 @@
           <parent link="base_link"/>
           <child link="belt12mm_base_link"/>
-          <origin xyz="2 0.5 0" rpy="0 0 1.57"/>
+          <origin xyz="2 -0.5 0" rpy="0 0 1.57"/>
   </joint>
 </robot>

Commit message: comment cout

File: urdf/camera_belt.urdf.xacro (robot description, xacro)
@@ -3,15 +3,15 @@
   <link name="base_link"/>
   <!-- d435i frame definition can be found at https://github.com/IntelRealSense/librealsense/blob/master/doc/d435i.md -->
-  <xacro:include filename="$(find realsense_gazebo_description)/urdf/_d435i.urdf.xacro" />
+  <!-- <xacro:include filename="$(find realsense_gazebo_description)/urdf/_d435i.urdf.xacro" />
   <xacro:sensor_d435i parent="base_link" name="camera" topics_ns="camera" visualize_color="true" align_depth="true" enable_pointCloud="true">
     <origin xyz="0.0 0.0 0.0" rpy="0.0 0.0 0.0"/>
-  </xacro:sensor_d435i>
+  </xacro:sensor_d435i> -->
   <!-- d405 -->
-  <!-- <xacro:include filename="$(find realsense2_description)/urdf/_d405.urdf.xacro" />
+  <xacro:include filename="$(find realsense2_description)/urdf/_d405.urdf.xacro" />
   <xacro:sensor_d405 parent="base_link" name="camera" topics_ns="camera" use_nominal_extrinsics="true" visualize_color="true" align_depth="true" enable_pointCloud="true">
     <origin xyz="0.0 0.0 0.0" rpy="0.0 0.0 0.0"/>
-  </xacro:sensor_d405> -->
+  </xacro:sensor_d405>
   <!-- add a belt10mm -->
-  <xacro:include filename="$(find belt10mm_description)/urdf/belt10mm.xacro"/>
+  <!-- <xacro:include filename="$(find belt10mm_description)/urdf/belt10mm.xacro"/>
   <xacro:belt10mm parent="base_link" prefix="belt10mm_">
     <origin xyz="0.0 0.0 0.0" rpy="0.0 0.0 0.0"/>
@@ -21,5 +21,5 @@
           <child link="belt10mm_base_link"/>
           <origin xyz="1 0.12 0" rpy="0 0 1.57"/>
-  </joint>
+  </joint> -->
   <!-- add a belt12mm -->
   <xacro:include filename="$(find belt12mm_description)/urdf/belt12mm.xacro"/>
@@ -30,5 +30,5 @@
           <parent link="base_link"/>
           <child link="belt12mm_base_link"/>
-          <origin xyz="1 -0.12 0" rpy="0 0 1.57"/>
+          <origin xyz="0.5 -0.12 0" rpy="0 0 1.57"/>
   </joint>
 </robot>
